File: placa_mestre/placa_mestre/placa_mestre.kicad_pcb (KiCad board)
At the start: 2 copper layers, 4 parts

Commit message: Add libs dos bornes, modelos 3D STEP dos ESP e organizada PCB
Parts:
- removed the REF** at (48.3, 61.0)
- removed the REF** at (218.4, 61.0)
- removed the REF** at (162.6, 61.0)
- added REF**: TE_1546216-3, 1546216-3:TE_1546216-3, F.Cu at (27.9, 43.2)
- added REF**: TE_1546216-3, 1546216-3:TE_1546216-3, F.Cu at (160.0, 121.9)
- added REF**: TE_1546216-3, 1546216-3:TE_1546216-3, F.Cu at (27.9, 91.4)
- added REF**: TE_1546216-3, 1546216-3:TE_1546216-3, F.Cu at (73.7, 58.4)
- added REF**: TE_1546216-3, 1546216-3:TE_1546216-3, F.Cu at (73.7, 91.4)
- added REF**: TE_1546216-3, 1546216-3:TE_1546216-3, F.Cu at (94.0, 27.9)
- added REF**: TE_1546216-2, 1546216-2:TE_1546216-2, F.Cu at (160.0, 71.1)
- added REF**: TE_1546216-2, 1546216-2:TE_1546216-2, F.Cu at (94.0, 134.6)
- added REF**: TE_1546216-2, 1546216-2:TE_1546216-2, F.Cu at (205.7, 134.6)
- added REF**: TE_1546216-3, 1546216-3:TE_1546216-3, F.Cu at (73.7, 121.9)
- added REF**: TE_1546216-3, 1546216-3:TE_1546216-3, F.Cu at (139.7, 91.4)
- added REF**: TE_1546216-3, 1546216-3:TE_1546216-3, F.Cu at (139.7, 27.9)
- added REF**: TE_1546216-3, 1546216-3:TE_1546216-3, F.Cu at (160.0, 43.2)
- added REF**: TE_1546216-2, 1546216-2:TE_1546216-2, F.Cu at (73.7, 134.6)
- added REF**: TE_1546216-3, 1546216-3:TE_1546216-3, F.Cu at (73.7, 106.7)
- added REF**: LoLin V3 NodeMCU, ESP8266:NodeMCU-LoLinV3, F.Cu at (116.8, 114.3)
- added REF**: TE_1546216-3, 1546216-3:TE_1546216-3, F.Cu at (139.7, 43.2)
- added REF**: TE_1546216-3, 1546216-3:TE_1546216-3, F.Cu at (160.0, 106.7)
- added REF**: TE_1546216-3, 1546216-3:TE_1546216-3, F.Cu at (27.9, 106.7)
- added REF**: TE_1546216-3, 1546216-3:TE_1546216-3, F.Cu at (73.7, 43.2)
- added REF**: TE_1546216-3, 1546216-3:TE_1546216-3, F.Cu at (94.0, 121.9)
- added REF**: TE_1546216-2, 1546216-2:TE_1546216-2, F.Cu at (27.9, 71.1)
- added REF**: TE_1546216-3, 1546216-3:TE_1546216-3, F.Cu at (94.0, 91.4)
- added REF**: TE_1546216-2, 1546216-2:TE_1546216-2, F.Cu at (205.7, 71.1)
- added REF**: TE_1546216-3, 1546216-3:TE_1546216-3, F.Cu at (205.7, 27.9)
- added REF**: TE_1546216-3, 1546216-3:TE_1546216-3, F.Cu at (27.9, 121.9)
- added REF**: TE_1546216-3, 1546216-3:TE_1546216-3, F.Cu at (205.7, 91.4)
- added REF**: TE_1546216-2, 1546216-2:TE_1546216-2, F.Cu at (94.0, 71.1)
- added REF**: TE_1546216-3, 1546216-3:TE_1546216-3, F.Cu at (160.0, 91.4)
- added REF**: LoLin V3 NodeMCU, ESP8266:NodeMCU-LoLinV3, F.Cu at (50.8, 114.3)
- added REF**: LoLin V3 NodeMCU, ESP8266:NodeMCU-LoLinV3, F.Cu at (182.9, 114.3)
- added REF**: TE_1546216-3, 1546216-3:TE_1546216-3, F.Cu at (160.0, 58.4)
- added REF**: TE_1546216-3, 1546216-3:TE_1546216-3, F.Cu at (160.0, 27.9)
- added REF**: TE_1546216-3, 1546216-3:TE_1546216-3, F.Cu at (27.9, 58.4)
- added REF**: LoLin V3 NodeMCU, ESP8266:NodeMCU-LoLinV3, F.Cu at (182.9, 50.8)
- added REF**: TE_1546216-2, 1546216-2:TE_1546216-2, F.Cu at (139.7, 71.1)
- added REF**: TE_1546216-2, 1546216-2:TE_1546216-2, F.Cu at (160.0, 134.6)
- added REF**: TE_1546216-2, 1546216-2:TE_1546216-2, F.Cu at (139.7, 134.6)
- added REF**: TE_1546216-3, 1546216-3:TE_1546216-3, F.Cu at (205.7, 43.2)
- added REF**: TE_1546216-3, 1546216-3:TE_1546216-3, F.Cu at (73.7, 27.9)
- added REF**: TE_1546216-3, 1546216-3:TE_1546216-3, F.Cu at (205.7, 58.4)
- added REF**: TE_1546216-3, 1546216-3:TE_1546216-3, F.Cu at (205.7, 121.9)
- added REF**: TE_1546216-3, 1546216-3:TE_1546216-3, F.Cu at (94.0, 106.7)
- added REF**: TE_1546216-3, 1546216-3:TE_1546216-3, F.Cu at (139.7, 106.7)
- added REF**: TE_1546216-3, 1546216-3:TE_1546216-3, F.Cu at (27.9, 27.9)
- added REF**: TE_1546216-3, 1546216-3:TE_1546216-3, F.Cu at (139.7, 121.9)
- added REF**: LoLin V3 NodeMCU, ESP8266:NodeMCU-LoLinV3, F.Cu at (50.8, 50.8)
- added REF**: TE_1546216-3, 1546216-3:TE_1546216-3, F.Cu at (205.7, 106.7)
- added REF**: TE_1546216-3, 1546216-3:TE_1546216-3, F.Cu at (139.7, 58.4)
- added REF**: TE_1546216-2, 1546216-2:TE_1546216-2, F.Cu at (73.7, 71.1)
- added REF**: TE_1546216-3, 1546216-3:TE_1546216-3, F.Cu at (94.0, 43.2)
- added REF**: TE_1546216-3, 1546216-3:TE_1546216-3, F.Cu at (94.0, 58.4)
- added REF**: TE_1546216-2, 1546216-2:TE_1546216-2, F.Cu at (27.9, 134.6)
- moved REF** 14.4 mm to (116.8, 50.8)
Other:
- board text added: "REF**"

Commit message: Add XL4005 volt. reg. to libs and PCB, also some traces.
Parts:
- added REF**: TE_1546216-3, 1546216-3:TE_1546216-3, F.Cu at (241.3, 71.1)
- added REF**: TE_1546216-3, 1546216-3:TE_1546216-3, F.Cu at (226.1, 71.1)
- added REF**: TE_1546216-3, 1546216-3:TE_1546216-3, F.Cu at (241.3, 106.7)
- added REF**: XL4005_DC-DC, XL4005:XL4005_DC-DC, F.Cu at (260.3, 17.6)
- added REF**: TE_1546216-3, 1546216-3:TE_1546216-3, F.Cu at (226.1, 106.7)
- added REF**: XL4005_DC-DC, XL4005:XL4005_DC-DC, F.Cu at (260.3, 114.1)
- added REF**: TE_1546216-3, 1546216-3:TE_1546216-3, F.Cu at (256.5, 106.7)
- added REF**: TE_1546216-3, 1546216-3:TE_1546216-3, F.Cu at (256.5, 71.1)
- added REF**: XL4005_DC-DC, XL4005:XL4005_DC-DC, F.Cu at (260.3, 43.0)
- added REF**: XL4005_DC-DC, XL4005:XL4005_DC-DC, F.Cu at (260.3, 139.5)
- moved REF** 3.59 mm to (157.5, 119.4)
- moved REF** 3.59 mm to (157.5, 68.6)
- moved REF** 3.59 mm to (157.5, 104.1)
- moved REF** 3.59 mm to (203.2, 68.6)
- moved REF** 3.59 mm to (203.2, 119.4)
- moved REF** 3.59 mm to (203.2, 104.1)
- moved REF** 3.59 mm to (203.2, 25.4)
- moved REF** 3.59 mm to (157.5, 25.4)
- moved REF** 3.59 mm to (157.5, 40.6)
- moved REF** 3.59 mm to (157.5, 55.9)
- moved REF** 3.59 mm to (203.2, 40.6)
- moved REF** 3.59 mm to (203.2, 55.9)
- moved REF** 3.59 mm to (91.4, 119.4)
- moved REF** 3.59 mm to (91.4, 68.6)
- moved REF** 3.59 mm to (91.4, 104.1)
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Routing:
- net (no net): track 0.00 -> 657.4 mm
Other:
- board text added: "12V+"
- board text added: "3.3V+"
- board text added: "5.0V+"
- board text added: "8.2V+"
- board text added: "9.0V+"
- board text added: "GND"
